File: pcb/firststep12.sch (KiCad schematic (older format))
At the start: 38 parts, among them SW1 SW_PUSH, SW10 SW_PUSH, SW11 SW_PUSH, SW12 SW_PUSH, SW13 SW_Push, SW2 SW_PUSH, SW3 SW_PUSH, SW4 SW_PUSH, SW5 SW_PUSH, SW6 SW_PUSH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

Commit message: create netlist
Parts:
- D1, D10, D11, D12, D2, D3, D4, D5, D6, D7, D8, D9: footprint (none) -> foostan:D3_TH
- L1, L10, L11, L12, L2, L3, L4, L5, L6, L7, L8, L9: footprint (none) -> foostan:SK6812MINI_rev
- SW1, SW10, SW11, SW12, SW2, SW3, SW4, SW5, SW6, SW7, SW8, SW9: footprint (none) -> foostan:CherryMX_1u
- SW13: footprint (none) -> foostan:ResetSW_1side
- U1: footprint (none) -> foostan:ProMicro_v3.5
Changed lines of the file:
@@
 F 0 "U1" H 1550 3137 60  0000 C CNN
 F 1 "ProMicro_r" H 1550 3031 60  0000 C CNN
-F 2 "" H 1650 1100 60  0000 C CNN
+F 2 "foostan:ProMicro_v3.5" H 1650 1100 60  0001 C CNN
 F 3 "" H 1650 1100 60  0000 C CNN
 	1    1500 2150
@@
 F 0 "SW2" H 4650 1505 50  0000 C CNN
 F 1 "SW_PUSH" H 4650 1414 50  0000 C CNN
-F 2 "" H 4650 1250 50  0000 C CNN
+F 2 "foostan:CherryMX_1u" H 4650 1250 50  0001 C CNN
 F 3 "" H 4650 1250 50  0000 C CNN
 	1    4650 1250
@@
 F 0 "SW3" H 5650 1505 50  0000 C CNN
 F 1 "SW_PUSH" H 5650 1414 50  0000 C CNN
-F 2 "" H 5650 1250 50  0000 C CNN
+F 2 "foostan:CherryMX_1u" H 5650 1250 50  0001 C CNN
 F 3 "" H 5650 1250 50  0000 C CNN
 	1    5650 1250
@@
 F 0 "SW4" H 6550 1505 50  0000 C CNN
 F 1 "SW_PUSH" H 6550 1414 50  0000 C CNN
-F 2 "" H 6550 1250 50  0000 C CNN
+F 2 "foostan:CherryMX_1u" H 6550 1250 50  0001 C CNN
 F 3 "" H 6550 1250 50  0000 C CNN
 	1    6550 1250
@@
 F 0 "D2" V 5096 1420 50  0000 R CNN
 F 1 "D" V 5005 1420 50  0000 R CNN
-F 2 "" H 5050 1500 50  0001 C CNN
+F 2 "foostan:D3_TH" H 5050 1500 50  0001 C CNN
 F 3 "~" H 5050 1500 50  0001 C CNN
 	1    5050 1500
@@
 F 0 "D3" V 6096 1420 50  0000 R CNN
 F 1 "D" V 6005 1420 50  0000 R CNN
-F 2 "" H 6050 1500 50  0001 C CNN
+F 2 "foostan:D3_TH" H 6050 1500 50  0001 C CNN
 F 3 "~" H 6050 1500 50  0001 C CNN
 	1    6050 1500
@@
 F 0 "D4" V 6996 1420 50  0000 R CNN
 F 1 "D" V 6905 1420 50  0000 R CNN
-F 2 "" H 6950 1500 50  0001 C CNN
+F 2 "foostan:D3_TH" H 6950 1500 50  0001 C CNN
 F 3 "~" H 6950 1500 50  0001 C CNN
 	1    6950 1500
@@
 F 0 "D1" V 4146 1420 50  0000 R CNN
 F 1 "D" V 4055 1420 50  0000 R CNN
-F 2 "" H 4100 1500 50  0001 C CNN
+F 2 "foostan:D3_TH" H 4100 1500 50  0001 C CNN
 F 3 "~" H 4100 1500 50  0001 C CNN
 	1    4100 1500
@@
 F 0 "SW1" H 3700 1505 50  0000 C CNN
 F 1 "SW_PUSH" H 3700 1414 50  0000 C CNN
-F 2 "" H 3700 1250 50  0000 C CNN
+F 2 "foostan:CherryMX_1u" H 3700 1250 50  0001 C CNN
 F 3 "" H 3700 1250 50  0000 C CNN
 	1    3700 1250
@@
 F 0 "SW5" H 3700 2355 50  0000 C CNN
 F 1 "SW_PUSH" H 3700 2264 50  0000 C CNN
-F 2 "" H 3700 2100 50  0000 C CNN
+F 2 "foostan:CherryMX_1u" H 3700 2100 50  0001 C CNN
 F 3 "" H 3700 2100 50  0000 C CNN
 	1    3700 2100
@@
 F 0 "SW6" H 4650 2355 50  0000 C CNN
 F 1 "SW_PUSH" H 4650 2264 50  0000 C CNN
-F 2 "" H 4650 2100 50  0000 C CNN
+F 2 "foostan:CherryMX_1u" H 4650 2100 50  0001 C CNN
 F 3 "" H 4650 2100 50  0000 C CNN
 	1    4650 2100
@@
 F 0 "SW7" H 5650 2355 50  0000 C CNN
 F 1 "SW_PUSH" H 5650 2264 50  0000 C CNN
-F 2 "" H 5650 2100 50  0000 C CNN
+F 2 "foostan:CherryMX_1u" H 5650 2100 50  0001 C CNN
 F 3 "" H 5650 2100 50  0000 C CNN
 	1    5650 2100
@@
 F 0 "SW8" H 6550 2355 50  0000 C CNN
 F 1 "SW_PUSH" H 6550 2264 50  0000 C CNN
-F 2 "" H 6550 2100 50  0000 C CNN
+F 2 "foostan:CherryMX_1u" H 6550 2100 50  0001 C CNN
 F 3 "" H 6550 2100 50  0000 C CNN
 	1    6550 2100
@@
 F 0 "D5" V 4146 2270 50  0000 R CNN
 F 1 "D" V 4055 2270 50  0000 R CNN
-F 2 "" H 4100 2350 50  0001 C CNN
+F 2 "foostan:D3_TH" H 4100 2350 50  0001 C CNN
 F 3 "~" H 4100 2350 50  0001 C CNN
 	1    4100 2350
@@
 F 0 "D6" V 5096 2270 50  0000 R CNN
 F 1 "D" V 5005 2270 50  0000 R CNN
-F 2 "" H 5050 2350 50  0001 C CNN
+F 2 "foostan:D3_TH" H 5050 2350 50  0001 C CNN
 F 3 "~" H 5050 2350 50  0001 C CNN
 	1    5050 2350
@@
 F 0 "D7" V 6096 2270 50  0000 R CNN
 F 1 "D" V 6005 2270 50  0000 R CNN
-F 2 "" H 6050 2350 50  0001 C CNN
+F 2 "foostan:D3_TH" H 6050 2350 50  0001 C CNN
 F 3 "~" H 6050 2350 50  0001 C CNN
 	1    6050 2350
@@
 F 0 "D8" V 6996 2270 50  0000 R CNN
 F 1 "D" V 6905 2270 50  0000 R CNN
-F 2 "" H 6950 2350 50  0001 C CNN
+F 2 "foostan:D3_TH" H 6950 2350 50  0001 C CNN
 F 3 "~" H 6950 2350 50  0001 C CNN
 	1    6950 2350
@@
 F 0 "SW9" H 3700 3105 50  0000 C CNN
 F 1 "SW_PUSH" H 3700 3014 50  0000 C CNN
-F 2 "" H 3700 2850 50  0000 C CNN
+F 2 "foostan:CherryMX_1u" H 3700 2850 50  0001 C CNN
 F 3 "" H 3700 2850 50  0000 C CNN
 	1    3700 2850
@@
 F 0 "SW10" H 4650 3105 50  0000 C CNN
 F 1 "SW_PUSH" H 4650 3014 50  0000 C CNN
-F 2 "" H 4650 2850 50  0000 C CNN
+F 2 "foostan:CherryMX_1u" H 4650 2850 50  0001 C CNN
 F 3 "" H 4650 2850 50  0000 C CNN
 	1    4650 2850
@@
 F 0 "SW11" H 5650 3105 50  0000 C CNN
 F 1 "SW_PUSH" H 5650 3014 50  0000 C CNN
-F 2 "" H 5650 2850 50  0000 C CNN
+F 2 "foostan:CherryMX_1u" H 5650 2850 50  0001 C CNN
 F 3 "" H 5650 2850 50  0000 C CNN
 	1    5650 2850
@@
 F 0 "SW12" H 6550 3105 50  0000 C CNN
 F 1 "SW_PUSH" H 6550 3014 50  0000 C CNN
-F 2 "" H 6550 2850 50  0000 C CNN
+F 2 "foostan:CherryMX_1u" H 6550 2850 50  0001 C CNN
 F 3 "" H 6550 2850 50  0000 C CNN
 	1    6550 2850
@@
 F 0 "D9" V 4146 3020 50  0000 R CNN
 F 1 "D" V 4055 3020 50  0000 R CNN
-F 2 "" H 4100 3100 50  0001 C CNN
+F 2 "foostan:D3_TH" H 4100 3100 50  0001 C CNN
 F 3 "~" H 4100 3100 50  0001 C CNN
 	1    4100 3100
@@
 F 0 "D10" V 5096 3020 50  0000 R CNN
 F 1 "D" V 5005 3020 50  0000 R CNN
-F 2 "" H 5050 3100 50  0001 C CNN
+F 2 "foostan:D3_TH" H 5050 3100 50  0001 C CNN
 F 3 "~" H 5050 3100 50  0001 C CNN
 	1    5050 3100
@@
 F 0 "D11" V 6096 3020 50  0000 R CNN
 F 1 "D" V 6005 3020 50  0000 R CNN
-F 2 "" H 6050 3100 50  0001 C CNN
+F 2 "foostan:D3_TH" H 6050 3100 50  0001 C CNN
 F 3 "~" H 6050 3100 50  0001 C CNN
 	1    6050 3100
@@
 F 0 "D12" V 6996 3020 50  0000 R CNN
 F 1 "D" V 6905 3020 50  0000 R CNN
-F 2 "" H 6950 3100 50  0001 C CNN
+F 2 "foostan:D3_TH" H 6950 3100 50  0001 C CNN
 F 3 "~" H 6950 3100 50  0001 C CNN
 	1    6950 3100
@@
 F 0 "L1" H 3400 3688 51  0000 C CNN
 F 1 "SK6812MINI" H 3400 3753 16  0000 C CNN
-F 2 "" H 3400 3950 60  0001 C CNN
+F 2 "foostan:SK6812MINI_rev" H 3400 3950 60  0001 C CNN
 F 3 "" H 3400 3950 60  0001 C CNN
 	1    3400 3950
@@
 F 0 "SW13" H 1550 3435 50  0000 C CNN
 F 1 "SW_Push" H 1550 3344 50  0000 C CNN
-F 2 "" H 1550 3350 50  0001 C CNN
+F 2 "foostan:ResetSW_1side" H 1550 3350 50  0001 C CNN
 F 3 "~" H 1550 3350 50  0001 C CNN
 	1    1550 3150
@@
 F 0 "L2" H 4000 3688 51  0000 C CNN
 F 1 "SK6812MINI" H 4000 3753 16  0000 C CNN
-F 2 "" H 4000 3950 60  0001 C CNN
+F 2 "foostan:SK6812MINI_rev" H 4000 3950 60  0001 C CNN
 F 3 "" H 4000 3950 60  0001 C CNN
 	1    4000 3950
@@
 F 0 "L3" H 4600 3688 51  0000 C CNN
 F 1 "SK6812MINI" H 4600 3753 16  0000 C CNN
-F 2 "" H 4600 3950 60  0001 C CNN
+F 2 "foostan:SK6812MINI_rev" H 4600 3950 60  0001 C CNN
 F 3 "" H 4600 3950 60  0001 C CNN
 	1    4600 3950
@@
 F 0 "L4" H 5200 3688 51  0000 C CNN
 F 1 "SK6812MINI" H 5200 3753 16  0000 C CNN
-F 2 "" H 5200 3950 60  0001 C CNN
+F 2 "foostan:SK6812MINI_rev" H 5200 3950 60  0001 C CNN
 F 3 "" H 5200 3950 60  0001 C CNN
 	1    5200 3950
@@
 F 0 "L5" H 5800 3688 51  0000 C CNN
 F 1 "SK6812MINI" H 5800 3753 16  0000 C CNN
-F 2 "" H 5800 3950 60  0001 C CNN
+F 2 "foostan:SK6812MINI_rev" H 5800 3950 60  0001 C CNN
 F 3 "" H 5800 3950 60  0001 C CNN
 	1    5800 3950
@@
 F 0 "L6" H 6400 3688 51  0000 C CNN
 F 1 "SK6812MINI" H 6400 3753 16  0000 C CNN
-F 2 "" H 6400 3950 60  0001 C CNN
+F 2 "foostan:SK6812MINI_rev" H 6400 3950 60  0001 C CNN
 F 3 "" H 6400 3950 60  0001 C CNN
 	1    6400 3950
@@
 F 0 "L7" H 3400 4438 51  0000 C CNN
 F 1 "SK6812MINI" H 3400 4503 16  0000 C CNN
-F 2 "" H 3400 4700 60  0001 C CNN
+F 2 "foostan:SK6812MINI_rev" H 3400 4700 60  0001 C CNN
 F 3 "" H 3400 4700 60  0001 C CNN
 	1    3400 4700
@@
 F 0 "L8" H 4000 4438 51  0000 C CNN
 F 1 "SK6812MINI" H 4000 4503 16  0000 C CNN
-F 2 "" H 4000 4700 60  0001 C CNN
+F 2 "foostan:SK6812MINI_rev" H 4000 4700 60  0001 C CNN
 F 3 "" H 4000 4700 60  0001 C CNN
 	1    4000 4700
@@
 F 0 "L9" H 4600 4438 51  0000 C CNN
 F 1 "SK6812MINI" H 4600 4503 16  0000 C CNN
-F 2 "" H 4600 4700 60  0001 C CNN
+F 2 "foostan:SK6812MINI_rev" H 4600 4700 60  0001 C CNN
 F 3 "" H 4600 4700 60  0001 C CNN
 	1    4600 4700
@@
 F 0 "L10" H 5200 4438 51  0000 C CNN
 F 1 "SK6812MINI" H 5200 4503 16  0000 C CNN
-F 2 "" H 5200 4700 60  0001 C CNN
+F 2 "foostan:SK6812MINI_rev" H 5200 4700 60  0001 C CNN
 F 3 "" H 5200 4700 60  0001 C CNN
 	1    5200 4700
@@
 F 0 "L11" H 5800 4438 51  0000 C CNN
 F 1 "SK6812MINI" H 5800 4503 16  0000 C CNN
-F 2 "" H 5800 4700 60  0001 C CNN
+F 2 "foostan:SK6812MINI_rev" H 5800 4700 60  0001 C CNN
 F 3 "" H 5800 4700 60  0001 C CNN
 	1    5800 4700
@@
 F 0 "L12" H 6400 4438 51  0000 C CNN
 F 1 "SK6812MINI" H 6400 4503 16  0000 C CNN
-F 2 "" H 6400 4700 60  0001 C CNN
+F 2 "foostan:SK6812MINI_rev" H 6400 4700 60  0001 C CNN
 F 3 "" H 6400 4700 60  0001 C CNN
 	1    6400 4700
