File: pcb/firststep12.kicad_pcb (KiCad board)
At the start: 2 copper layers, 89.2 x 99.6 mm, 44 parts, among them SW1 SW_PUSH, SW10 SW_PUSH, SW11 SW_PUSH, SW12 SW_PUSH, SW13 SW_Push, SW2 SW_PUSH, SW3 SW_PUSH, SW4 SW_PUSH, SW5 SW_PUSH, SW6 SW_PUSH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

Commit message: add gerber, bottom plate, top plate
Routing:
- net VCC: track 312.1 -> 313.9 mm
Other:
- board size 89.2 x 99.6 mm -> 87.2 x 99.6 mm
